File: board/board.kicad_sch (KiCad schematic)
At the start: 6 parts, among them J1 TFDU4101

Commit message: 20230413_081659
Parts:
- removed C1: 4.7uF 16V, symbol Device:C_Polarized_US
- removed C?: 0.1uF 16V, symbol Device:C
- removed J1: TFDU4101, symbol Connector:Conn_01x08_Female
- removed R1: 56R, symbol Device:R
- removed R?: 47R, symbol Device:R
- removed U?: STM32H750VBTx, Package_QFP:LQFP-100_14x14mm_P0.5mm, symbol MCU_ST_STM32H7:STM32H750VBTx
Connections:
- no-connect marks 2 -> 0
Other:
- company: (none) -> Developed by Molganov A.A
- title: (none) -> OptiREX_DevBoard

Commit message: 20230413_082240
Other:
- title: OptiREX_DevBoard -> ProjectOptics_DevBoard
Changed lines of the file:
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@@
   (paper "A4")
   (title_block
-    (title "OptiREX_DevBoard")
+    (title "ProjectOptics_DevBoard")
     (date "2023-03-26")
     (rev "5")
